File: hardware/flash_adapter/flash_adapter.kicad_pcb (KiCad board)
At the start: 2 copper layers, 13 x 22 mm, 2 parts, among them J1 FTSH-105-01-L-DV-K-TR, J2 HX PZ2.54-2x5P WT

Commit message: Add flash adapter silkscreen logo
Parts:
- added G***: LOGO, schneggi_library:schneggi, B.Cu at (18.5, 29.5)
